Commit message: the description of the robot model is close to the real one; added map saver launch and localization config

File: kitty_description/urdf/params.urdf.xacro (robot description, xacro)
@@ -4,17 +4,17 @@
     <xacro:property name="yaml_file" value="$(find kitty_description)/config/props.yaml" />
     <xacro:property name="props" value="${xacro.load_yaml(yaml_file)}" />
-    <xacro:property name="front_wheel_2_front_bumper" value="0.1" />
-    <xacro:property name="rear_wheel_2_rear_bumper" value="0.1" />
+    <xacro:property name="front_wheel_2_front_bumper" value="0.05" />
+    <xacro:property name="rear_wheel_2_rear_bumper" value="0.05" />
     <xacro:property name="wheelbase" value="${props['wheelbase']}" />
     <xacro:property name="track_width" value="${props['track_width']}" />
     <!-- основные габариты -->
     <xacro:property name="body_length" value="${front_wheel_2_front_bumper+wheelbase+rear_wheel_2_rear_bumper}" />
-    <xacro:property name="body_width" value="0.8" />
-    <xacro:property name="body_heigth" value="0.8" />
-    <xacro:property name="body_mass" value="0.1" />
+    <xacro:property name="body_width" value="0.5" />
+    <xacro:property name="body_heigth" value="0.5" />
+    <xacro:property name="body_mass" value="7.0" />
     <!-- габариты колес -->
     <xacro:property name="wheel_width" value="0.025" />
     <xacro:property name="wheel_radius" value="${props['wheel_radius']}" />
-    <xacro:property name="wheel_mass" value="0.02" />
+    <xacro:property name="wheel_mass" value="0.1" />
     <xacro:property name="wheel_turn_limit" value="${pi/4}" />
     <xacro:property name="wheel_shift_z" value="0.0" /> <!-- расстояние по оси Z между передней осью и осью вращения колеса -->
