Commit message: add real kitty config in sim

File: kitty_description/urdf/base.urdf.xacro (robot description, xacro)
@@ -71,20 +71,20 @@
 		prefix="rear_right"
 		parent="rear_axis_link"
-		steer_origin_xyz="0 -${track_width/2} 0"
+		steer_origin_xyz="0 -${track_width/2} -${wheel_suspension}"
 		steer_limit="${wheel_turn_limit}" />
 	<xacro:steer_wheel
 		prefix="rear_left"
 		parent="rear_axis_link"
-		steer_origin_xyz="0 ${track_width/2} 0"
+		steer_origin_xyz="0 ${track_width/2} -${wheel_suspension}"
 		steer_limit="${wheel_turn_limit}" />
 	<xacro:steer_wheel
 		prefix="front_right"
 		parent="front_axis_link"
-		steer_origin_xyz="0 -${track_width/2} 0"
+		steer_origin_xyz="0 -${track_width/2} -${wheel_suspension}"
 		steer_limit="${wheel_turn_limit}" />
 	<xacro:steer_wheel
 		prefix="front_left"
 		parent="front_axis_link"
-		steer_origin_xyz="0 ${track_width/2} 0"
+		steer_origin_xyz="0 ${track_width/2} -${wheel_suspension}"
 		steer_limit="${wheel_turn_limit}" />
 	<!-- gazebo plugins -->

File: kitty_description/urdf/config.urdf.xacro (robot description, xacro)
@@ -8,5 +8,5 @@
 		prefix="bottom"
 		parent="base_link"
-		origin_xyz="0.0 0.0 -${wheel_radius/2}"
+		origin_xyz="-0.15 0.0 -0.043"
 		origin_rpy="3.14159 0.0 0.0" />
 	<xacro:rs_camera

File: kitty_description/urdf/params.urdf.xacro (robot description, xacro)
@@ -4,18 +4,18 @@
     <xacro:property name="yaml_file" value="$(find kitty_description)/config/props.yaml" />
     <xacro:property name="props" value="${xacro.load_yaml(yaml_file)}" />
-    <xacro:property name="front_wheel_2_front_bumper" value="0.05" />
-    <xacro:property name="rear_wheel_2_rear_bumper" value="0.05" />
+    <xacro:property name="front_wheel_2_front_bumper" value="0.04" />
+    <xacro:property name="rear_wheel_2_rear_bumper" value="0.04" />
     <xacro:property name="wheelbase" value="${props['wheelbase']}" />
     <xacro:property name="track_width" value="${props['track_width']}" />
     <!-- основные габариты -->
     <xacro:property name="body_length" value="${front_wheel_2_front_bumper+wheelbase+rear_wheel_2_rear_bumper}" />
-    <xacro:property name="body_width" value="0.5" />
-    <xacro:property name="body_heigth" value="0.5" />
+    <xacro:property name="body_width" value="0.42" />
+    <xacro:property name="body_heigth" value="0.275" />
     <xacro:property name="body_mass" value="7.0" />
     <!-- габариты колес -->
-    <xacro:property name="wheel_width" value="0.025" />
+    <xacro:property name="wheel_width" value="0.027" />
     <xacro:property name="wheel_radius" value="${props['wheel_radius']}" />
     <xacro:property name="wheel_mass" value="0.1" />
     <xacro:property name="wheel_turn_limit" value="${pi/4}" />
-    <xacro:property name="wheel_shift_z" value="0.0" /> <!-- расстояние по оси Z между передней осью и осью вращения колеса -->
+    <xacro:property name="wheel_suspension" value="0.07" /> <!-- расстояние по оси Z между передней осью и осью вращения колеса -->
 </robot>

Commit message: updated the urdf model according to the updated macros (suspension_height was added to the wheels and the base was added to the lidar)

File: kitty_description/urdf/base.urdf.xacro (robot description, xacro)
@@ -16,5 +16,5 @@
 		<parent link="base_footprint" />
 		<child link="base_link" />
-		<origin xyz="0 0 ${wheel_radius}" rpy="0 0 0" />
+		<origin xyz="0 0 ${wheel_radius + suspension_height}" rpy="0 0 0" />
 	</joint>
 	<link name="base_link">
@@ -71,21 +71,25 @@
 		prefix="rear_right"
 		parent="rear_axis_link"
-		steer_origin_xyz="0 -${track_width/2} -${wheel_suspension}"
-		steer_limit="${wheel_turn_limit}" />
+		suspension_origin_xyz="0 -${track_width/2} 0"
+		suspension_height="${suspension_height}"
+		steer_limit="${steer_limit}" />
 	<xacro:steer_wheel
 		prefix="rear_left"
 		parent="rear_axis_link"
-		steer_origin_xyz="0 ${track_width/2} -${wheel_suspension}"
-		steer_limit="${wheel_turn_limit}" />
+		suspension_origin_xyz="0 ${track_width/2} 0"
+		suspension_height="${suspension_height}"
+		steer_limit="${steer_limit}" />
 	<xacro:steer_wheel
 		prefix="front_right"
 		parent="front_axis_link"
-		steer_origin_xyz="0 -${track_width/2} -${wheel_suspension}"
-		steer_limit="${wheel_turn_limit}" />
+		suspension_origin_xyz="0 -${track_width/2} 0"
+		suspension_height="${suspension_height}"
+		steer_limit="${steer_limit}" />
 	<xacro:steer_wheel
 		prefix="front_left"
 		parent="front_axis_link"
-		steer_origin_xyz="0 ${track_width/2} -${wheel_suspension}"
-		steer_limit="${wheel_turn_limit}" />
+		suspension_origin_xyz="0 ${track_width/2} 0"
+		suspension_height="${suspension_height}"
+		steer_limit="${steer_limit}" />
 	<!-- gazebo plugins -->
 	<gazebo>

File: kitty_description/urdf/config.urdf.xacro (robot description, xacro)
@@ -8,5 +8,5 @@
 		prefix="bottom"
 		parent="base_link"
-		origin_xyz="-0.15 0.0 -0.043"
+		origin_xyz="-0.15 0.0 0.0"
 		origin_rpy="3.14159 0.0 0.0" />
 	<xacro:rs_camera

File: kitty_description/urdf/params.urdf.xacro (robot description, xacro)
@@ -4,18 +4,19 @@
     <xacro:property name="yaml_file" value="$(find kitty_description)/config/props.yaml" />
     <xacro:property name="props" value="${xacro.load_yaml(yaml_file)}" />
+    <!-- основные габариты -->
+    <xacro:property name="wheelbase" value="${props['wheelbase']}" />
+    <xacro:property name="track_width" value="${props['track_width']}" />
     <xacro:property name="front_wheel_2_front_bumper" value="0.04" />
     <xacro:property name="rear_wheel_2_rear_bumper" value="0.04" />
-    <xacro:property name="wheelbase" value="${props['wheelbase']}" />
-    <xacro:property name="track_width" value="${props['track_width']}" />
-    <!-- основные габариты -->
     <xacro:property name="body_length" value="${front_wheel_2_front_bumper+wheelbase+rear_wheel_2_rear_bumper}" />
     <xacro:property name="body_width" value="0.42" />
     <xacro:property name="body_heigth" value="0.275" />
     <xacro:property name="body_mass" value="7.0" />
-    <!-- габариты колес -->
+    <!-- характеристики колес -->
     <xacro:property name="wheel_width" value="0.027" />
     <xacro:property name="wheel_radius" value="${props['wheel_radius']}" />
     <xacro:property name="wheel_mass" value="0.1" />
-    <xacro:property name="wheel_turn_limit" value="${pi/4}" />
-    <xacro:property name="wheel_suspension" value="0.07" /> <!-- расстояние по оси Z между передней осью и осью вращения колеса -->
+    <!-- характеристики подвески -->
+    <xacro:property name="steer_limit" value="${pi/4}" />
+    <xacro:property name="suspension_height" value="0.07" />
 </robot>

Commit message: removed front_ and rear_axis

File: kitty_description/urdf/base.urdf.xacro (robot description, xacro)
@@ -43,51 +43,27 @@
 		<selfCollide>false</selfCollide>
 	</gazebo>
-	<!-- REAR AXIS LINK -->
-	<joint name="base_link_2_rear_axis_link" type="fixed">
-		<parent link="base_link" />
-		<child link="rear_axis_link" />
-		<origin xyz="${-(body_length/2-rear_wheel_2_rear_bumper)} 0 0" rpy="0 0 0" />
-	</joint>
-	<link name="rear_axis_link">
-		<xacro:null_visual/>
-		<xacro:null_collision/>
-		<xacro:null_inertia/>
-	</link>
-	<gazebo reference="rear_axis_link" />
-	<!-- FRONT AXIS LINK -->
-	<joint name="base_link_2_front_axis_link" type="fixed">
-		<parent link="base_link" />
-		<child link="front_axis_link" />
-		<origin xyz="${body_length/2-front_wheel_2_front_bumper} 0 0" rpy="0 0 0" />
-	</joint>
-	<link name="front_axis_link">
-		<xacro:null_visual/>
-		<xacro:null_collision/>
-		<xacro:null_inertia/>
-	</link>
-	<gazebo reference="front_axis_link" />
 	<!-- WHEELS -->
 	<xacro:steer_wheel
 		prefix="rear_right"
-		parent="rear_axis_link"
-		suspension_origin_xyz="0 -${track_width/2} 0"
+		parent="base_link"
+		suspension_origin_xyz="${-(body_length/2-rear_wheel_2_rear_bumper)} -${track_width/2} 0"
 		suspension_height="${suspension_height}"
 		steer_limit="${steer_limit}" />
 	<xacro:steer_wheel
 		prefix="rear_left"
-		parent="rear_axis_link"
-		suspension_origin_xyz="0 ${track_width/2} 0"
+		parent="base_link"
+		suspension_origin_xyz="${-(body_length/2-rear_wheel_2_rear_bumper)} ${track_width/2} 0"
 		suspension_height="${suspension_height}"
 		steer_limit="${steer_limit}" />
 	<xacro:steer_wheel
 		prefix="front_right"
-		parent="front_axis_link"
-		suspension_origin_xyz="0 -${track_width/2} 0"
+		parent="base_link"
+		suspension_origin_xyz="${body_length/2-front_wheel_2_front_bumper} -${track_width/2} 0"
 		suspension_height="${suspension_height}"
 		steer_limit="${steer_limit}" />
 	<xacro:steer_wheel
 		prefix="front_left"
-		parent="front_axis_link"
-		suspension_origin_xyz="0 ${track_width/2} 0"
+		parent="base_link"
+		suspension_origin_xyz="${body_length/2-front_wheel_2_front_bumper} ${track_width/2} 0"
 		suspension_height="${suspension_height}"
 		steer_limit="${steer_limit}" />
